File: hw/controller/PhoneController.kicad_pcb (KiCad board)
At the start: 2 copper layers, 62 x 47 mm, 58 parts, among them J1 Conn_01x03_Pin, J2 52746-0671, SW1 SW_Push, SW10 SW_Push, SW11 SW_Push, SW12 SW_Push, SW13 SW_Push, SW14 SW_Push, SW2 SW_Push, SW3 SW_Push, SW4 SW_Push, SW5 SW_Push, SW6 SW_Push, SW7 SW_Push, SW8 SW_Push, SW9 SW_Push, U1 RP2040, U3 AMS1117-3.3, U4 W25Q128JVS, Y1 Crystal_GND24

Commit message: chore: Updating schematics
Parts:
- added R21: 5.1k Ohm, Resistor_SMD:R_0805_2012Metric_Pad1.20x1.40mm_HandSolder, B.Cu at (43.3, 41.5)
- SW1, SW10: moved to F.Cu
- SW11, SW12, SW13, SW14, SW2, SW3, SW4, SW5, SW6, SW7, SW8, SW9: moved to B.Cu
- moved R3 50.0 mm to (55.9, 24.9), turned to 0 degrees
- moved SW3 50.0 mm to (56.0, 22.4), turned to 0 degrees
- moved SW4 45.2 mm to (8.40, 22.5), turned to 0 degrees
- moved R4 45.1 mm to (8.63, 25.0)
- moved U4 39.1 mm to (16.8, 3.17)
- moved J2 36.6 mm to (49.6, 40.3)
- moved R10 36.6 mm to (51.2, 36.6)
- moved R11 36.6 mm to (49.1, 36.6)
- moved SW2 35.0 mm to (48.5, 15.0)
- moved SW6 35.0 mm to (48.5, 30.0)
- moved R6 32.2 mm to (45.6, 29.9)
- moved R2 32.0 mm to (45.5, 14.7)
- moved R18 31.3 mm to (18.4, 15.1), turned to 180 degrees
- moved C14 25.6 mm to (20.4, 25.3)
- moved U1 25.6 mm to (26.7, 32.0)
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Routing:
- net BTN_SR: track 155.7 -> 66.4 mm, vias 4 -> 2
- net BTN_X: track 50.2 -> 128.8 mm, vias 2 -> 4
- net BTN_Y: track 75.3 -> 140.8 mm
- net BTN_SL: track 90.9 -> 129.9 mm, vias 4 -> 2
- net QSPI_SCLK: track 4.16 -> 39.0 mm, vias 0 -> 2
- net QSPI_SD3: track 3.80 -> 38.2 mm, vias 0 -> 2
- net QSPI_SD0: track 4.52 -> 38.8 mm, vias 0 -> 2
- net BTN_DN: track 62.6 -> 32.7 mm
- net SWD: track 9.15 -> 38.0 mm, vias 1 -> 2
- net BTN_RT: track 49.5 -> 21.0 mm
- net BTN_A: track 22.0 -> 50.3 mm, vias 1 -> 4
- net BTN_SLCT: track 32.8 -> 6.86 mm, vias 1 -> 0
- net SWCLK: track 13.4 -> 39.0 mm, vias 1 -> 2
- net QSPI_SD2: track 13.0 -> 37.6 mm, vias 0 -> 2
- net 3.3v: track 178.8 -> 202.5 mm, vias 17 -> 22
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Other:
- outline, holes or cut-outs redrawn
- board text added: "JoyFon v0.4"
- board text added: "Rst"
- board text removed: "D+"
- board text removed: "D-"
- board text removed: "JoyFon v0.3"
- board text removed: "RESET"
