File: hw/controller/PhoneController.kicad_sch (KiCad schematic)
At the start: 57 parts, among them J1 Conn_01x03_Pin, J2 52746-0671, SW1 SW_Push, SW10 SW_Push, SW11 SW_Push, SW12 SW_Push, SW13 SW_Push, SW14 SW_Push, SW2 SW_Push, SW3 SW_Push, SW4 SW_Push, SW5 SW_Push, SW6 SW_Push, SW7 SW_Push, SW8 SW_Push, SW9 SW_Push, U1 RP2040, U3 AMS1117-3.3, U4 W25Q128JVS, Y1 Crystal_GND24

Commit message: chore: Updating schematics
Parts:
- added R21: 5.1k Ohm, Resistor_SMD:R_0805_2012Metric_Pad1.20x1.40mm_HandSolder, symbol Device:R
Connections:
- net CC2: now also R21.1
- net GND: now also R21.2
Other:
- moved on the sheet: R19, R20, SW13, SW14
