File: hw/usb/PhoneControllerUSB.kicad_sch (KiCad schematic)
At the start: 2 parts, among them J1 525590652, J2 DX07VN24WA2C1568

Commit message: chore: Updating schematics
Parts:
- J1: footprint 52559-0652:CON_525590652_MOL -> 52746-0671:52746-0671
- J2: footprint DX07VN24WA2C1568:DX07VN24WA2C1568 -> Type-C-31-M-12:USBC1-AM-063
Changed lines of the file:
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@@
 (kicad_sch
-	(version 20231120)
+	(version 20250114)
 	(generator "eeschema")
-	(generator_version "8.0")
+	(generator_version "9.0")
 	(paper "A4")
 	(no_connect
@@
 			)
 		)
-		(property "Footprint" "DX07VN24WA2C1568:DX07VN24WA2C1568"
+		(property "Footprint" "Type-C-31-M-12:USBC1-AM-063"
 			(at 140.97 126.67 0)
 			(effects
@@
 			)
 		)
-		(property "Footprint" "52559-0652:CON_525590652_MOL"
+		(property "Footprint" "52746-0671:52746-0671"
 			(at 77.47 40.64 0)
 			(effects
@@
 		)
 	)
+	(embedded_fonts no)
 )
